File: raspi3-4xMCP2517FD.sch (KiCad schematic (older format))
At the start: 44 parts, among them J1 Raspberry_Pi_2_3, J2 Conn_02x04_Odd_Even, U1 MCP2517FD-xSL, U2 MCP2517FD-xSL, U3 MCP2517FD-xSL, U4 MCP2517FD-xSL, U5 TJA1049T-3, U6 TJA1049T-3, U7 TJA1049T-3, U8 TJA1049T-3, X1 ASV-20MHz

Commit message: make v2
Parts:
- removed R5, R7, R9: 10K, Resistor_SMD:R_0603_1608Metric, symbol Device:R
- added C22: 100nF, Capacitor_SMD:C_0603_1608Metric, symbol Device:C_Small
- added R1, R2: 3K9, Resistor_SMD:R_0603_1608Metric, symbol Device:R
- added R13, R14: dnp, Capacitor_SMD:C_0805_2012Metric, symbol Device:R
- added R3: 10K, Resistor_SMD:R_0603_1608Metric, symbol Device:R
- added U9: AT24CS32-SSHM, Package_SO:SOIC-8_3.9x4.9mm_P1.27mm, symbol Memory_EEPROM:AT24CS32-SSHM
- R11, R12: value 10K -> dnp; footprint Resistor_SMD:R_0603_1608Metric -> Capacitor_SMD:C_0805_2012Metric
- renumbered C2 to C1, C14 to C11, C7 to C12, C11 to C13, C15 to C14, C8 to C15, C12 to C16, C16 to C17, C9 to C18, C13 to C19, C18 to C2, C17 to C20, C1 to C21, C19 to C4, C4 to C5, C20 to C6, C5 to C7, C21 to C8, C6 to C9, R2 to R5, R3 to R7, R1 to R9
Connections:
- net labels added: ID_SC, ID_SD
- net labels removed: MCP0_INT0, MCP0_INT1, MCP1_INT0, MCP1_INT1, MCP2_INT0, MCP2_INT1, MCP3_INT0, MCP3_INT1
- wire segments 61 -> 121
- no-connect marks 15 -> 25
